File: kicad/LED_Chain.kicad_sch (KiCad schematic)
At the start: 33 parts, among them J1 Interface, J2 PWR, J3 NeoPixel R1 A, J4 NeoPixel R1 B, J5 NeoPixel R1 C, J6 NeoPixel R1 D, J7 LED, Q1 IRLML2502, Q2 IRLML2502, Q3 IRLML2502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

Commit message: Updated for V8 KiCad
Parts:
- U1: footprint Package_SO:SOIC-16_3.9x9.9mm_P1.27mm -> LED_Chain:SO-16-N
Changed lines of the file:
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@@
 			)
 		)
-		(property "Footprint" "Package_SO:SOIC-16_3.9x9.9mm_P1.27mm"
+		(property "Footprint" "LED_Chain:SO-16-N"
 			(at 60.96 54.61 0)
 			(effects
@@
 			)
 		)
-		(property "Footprint" "Package_SO:SOIC-16_3.9x9.9mm_P1.27mm"
+		(property "Footprint" "LED_Chain:SO-16-N"
 			(at 162.56 137.16 0)
 			(effects
@@
 			)
 		)
-		(property "Footprint" "Package_SO:SOIC-16_3.9x9.9mm_P1.27mm"
+		(property "Footprint" "LED_Chain:SO-16-N"
 			(at 162.56 110.49 0)
 			(effects
